Commit message: update gazebo simulation

File: ws_robot/src/robot/ned_ros/niryo_robot_description/urdf/one/niryo_one_gazebo.urdf.xacro (robot description, xacro)
@@ -8,5 +8,6 @@
     </gazebo>
     <!-- Import Robot -->
-    <xacro:include filename="$(find niryo_robot_description)/urdf/one/niryo_one.urdf.xacro"/>
+    <!-- <xacro:include filename="$(find niryo_robot_description)/urdf/one/niryo_one.urdf.xacro"/> -->
+ <xacro:include filename="$(find niryo_one_urdf)/niryo_one.urdf.xacro"/>
     <!-- Import Transmission -->
     <xacro:include filename="$(find niryo_robot_description)/urdf/one/niryo_one.transmission.xacro"/>

File: ws_robot/src/robot/niryo_one_urdf/niryo_one.urdf.xacro (robot description, xacro)
@@ -28,4 +28,5 @@
     <xacro:property name="distance_hand_tool" value="0.0073" />
 	<xacro:property name="PI" value="3.14159265359" />
+    <xacro:property name="deg_to_rad" value="${PI/180}"/>
     <xacro:property name="limit_low_shoulder_rotation" value="-3.05433" />
     <xacro:property name="limit_up_shoulder_rotation" value="3.05433" />
@@ -55,4 +56,9 @@
             </geometry>
         </collision>
+        <inertial>
+            <origin xyz="0 0 ${distance_origin_shoulder_z / 2}" rpy="0 0 0"/>
+            <mass value="1.2"/>
+            <inertia ixx="0.0015" ixy="0.0" ixz="0.0" iyy="0.0015" iyz="0.0" izz="0.0015"/>
+        </inertial>
 	</link>
     <link name="shoulder_link">
@@ -69,4 +75,9 @@
             </geometry>
         </collision>
+        <inertial>
+            <origin xyz="0 0 ${distance_shoulder_arm_z / 2}" rpy="0 0 0"/>
+            <mass value="0.8"/>
+            <inertia ixx="0.0015" ixy="0.0" ixz="0.0" iyy="0.0015" iyz="0.0" izz="0.0015"/>
+        </inertial>
 	</link>
     <link name="arm_link">
@@ -83,4 +94,9 @@
             </geometry>
         </collision>
+                <inertial>
+            <origin xyz="${distance_arm_elbow_x / 2} -0.1 0" rpy="0 0 0"/>
+            <mass value="0.4"/>
+            <inertia ixx="0.0015" ixy="0.0" ixz="0.0" iyy="0.0015" iyz="0.0" izz="0.0015"/>
+        </inertial>
 	</link>
     <link name="elbow_link">
@@ -97,4 +113,9 @@
             </geometry>
         </collision>
+                <inertial>
+            <origin xyz="${distance_elbow_forearm_x / 2} ${distance_elbow_forearm_y / 2} 0" rpy="0 0 0"/>
+            <mass value="0.3"/>
+            <inertia ixx="0.0015" ixy="0.0" ixz="0.0" iyy="0.0015" iyz="0.0" izz="0.0015"/>
+        </inertial>
 	</link>
     <link name="forearm_link">
@@ -111,4 +132,9 @@
             </geometry>
         </collision>
+                <inertial>
+            <origin xyz="0 0 ${distance_forearm_wrist_z / 2}" rpy="0 0 0"/>
+            <mass value="0.3"/>
+            <inertia ixx="0.0015" ixy="0.0" ixz="0.0" iyy="0.0015" iyz="0.0" izz="0.0015"/>
+        </inertial>
 	</link>
     <link name="wrist_link">
@@ -125,4 +151,9 @@
             </geometry>
         </collision>
+        <inertial>
+            <origin xyz="${distance_wrist_hand_x / 2} ${distance_wrist_hand_y / 2} 0" rpy="0 0 0"/>
+            <mass value="0.15"/>
+            <inertia ixx="0.001" ixy="0.0" ixz="0.0" iyy="0.001" iyz="0.0" izz="0.001"/>
+        </inertial>
 	</link>
     <link name="hand_link">
@@ -139,4 +170,9 @@
             </geometry>
         </collision>
+        <inertial>
+            <origin xyz="0 0 ${distance_hand_tool / 2}" rpy="0 0 0"/>
+            <mass value="0.05"/>
+            <inertia ixx="0.001" ixy="0.0" ixz="0.0" iyy="0.001" iyz="0.0" izz="0.001"/>
+        </inertial>
 	</link>
     <link name="tool_link">
@@ -154,4 +190,5 @@
 		<axis xyz="0 0 1" />
 		<limit effort="1" velocity="1.0" lower="${limit_low_shoulder_rotation}" upper="${limit_up_shoulder_rotation}" />
+        <dynamics damping="0.1" friction="0.0"/>
 	</joint>
 	<joint name="joint_2" type="revolute">
@@ -161,4 +198,5 @@
 		<limit effort="1" velocity="1.0" lower="${limit_low_arm_rotation}" upper="${limit_up_arm_rotation}" />
 		<axis xyz="0 0 1" />
+        <dynamics damping="0.1" friction="0.0"/>
 	</joint>
 	<joint name="joint_3" type="revolute">
@@ -168,4 +206,5 @@
 		<limit effort="1" velocity="1.0" lower="${limit_low_elbow_rotation}" upper="${limit_up_elbow_rotation}" />
 		<axis xyz="0 0 1" />
+         <dynamics damping="0.1" friction="0.0"/>
 	</joint>
 	<joint name="joint_4" type="revolute">
@@ -175,4 +214,5 @@
 		<limit effort="1" velocity="1.0" lower="${limit_low_forearm_rotation}" upper="${limit_up_forearm_rotation}" />
 		<axis xyz="0 0 1" />
+         <dynamics damping="0.1" friction="0.0"/>
 	</joint>
 	<joint name="joint_5" type="revolute">
@@ -182,4 +222,5 @@
 		<limit effort="1" velocity="1.0" lower="${limit_low_wrist_rotation}" upper="${limit_up_wrist_rotation}" />
 		<axis xyz="0 0 1" />
+         <dynamics damping="0.1" friction="0.0"/>
 	</joint>
 	<joint name="joint_6" type="revolute">
@@ -189,4 +230,5 @@
 		<limit effort="1" velocity="1.0" lower="${limit_low_hand_rotation}" upper="${limit_up_hand_rotation}" />
 		<axis xyz="0 0 1" />
+         <dynamics damping="0.1" friction="0.0"/>
 	</joint>
 	<joint name="hand_tool_joint" type="fixed">
