Commit message: update test2.launch

File: ws_robot/src/robot/ned_ros/niryo_robot_description/urdf/one/niryo_one.urdf.xacro (robot description, xacro)
@@ -153,5 +153,5 @@
         <parent link="world"/>
         <child link="base_link"/>
-        <origin xyz="0 0 0" rpy="0 0 0"/>
+        <origin xyz="0 0 0.63" rpy="0 0 0"/>
     </joint>
     <joint name="joint_1" type="revolute">

File: ws_robot/src/robot/ned_ros/niryo_robot_description/urdf/one/niryo_one_camera.urdf.xacro (robot description, xacro)
@@ -27,5 +27,4 @@
                 <box size="${cameraWidth} ${cameraWidth} ${cameraHeight}"/>
             </geometry>
-            <material name="DarkGrey"/>
         </visual>
         <inertial>

File: ws_robot/src/robot/ned_ros/niryo_robot_description/urdf/one/niryo_one_gazebo.urdf.xacro (robot description, xacro)
@@ -9,5 +9,5 @@
     <!-- Import Robot -->
     <!-- <xacro:include filename="$(find niryo_robot_description)/urdf/one/niryo_one.urdf.xacro"/> -->
- <xacro:include filename="$(find niryo_one_urdf)/niryo_one.urdf.xacro"/>
+    <xacro:include filename="$(find niryo_robot_description)/urdf/one/niryo_one.urdf.xacro"/>
     <!-- Import Transmission -->
     <xacro:include filename="$(find niryo_robot_description)/urdf/one/niryo_one.transmission.xacro"/>

File: ws_robot/src/robot/ned_ros/niryo_robot_description/urdf/one/niryo_one_gripper_gazebo.urdf.xacro (robot description, xacro)
@@ -1,16 +1,5 @@
 <?xml version="1.0"?>
 <robot xmlns:xacro="http://www.ros.org/wiki/xacro" name="niryo_one">
-    <!-- <xacro:include filename="$(find niryo_robot_description)/urdf/one/niryo_one_camera.urdf.xacro"/> -->
- <xacro:include filename="$(find niryo_robot_description)/urdf/one/niryo_one_gazebo.urdf.xacro"/>
-    <!-- gazebo joint state publisher for all joints. Necessary to control mors -->
-    <gazebo>
-        <plugin name="passive_joint_state_publisher" filename="libgazebo_ros_joint_state_publisher.so">
-            <jointName>joint_1, joint_2, joint_3, joint_4, joint_5, joint_6,
-                joint_base_to_mors_1, joint_base_to_mors_2
-            </jointName>
-            <updateRate>50.0</updateRate>
-            <alwaysOn>true</alwaysOn>
-        </plugin>
-    </gazebo>
+    <xacro:include filename="$(find niryo_robot_description)/urdf/one/niryo_one_gazebo.urdf.xacro"/>
     <!-- Joint from tool_link to base_gripper -->
     <joint name="joint_to_gripper" type="fixed">
@@ -145,6 +134,6 @@
     </joint>
     <!-- Transmissions -->
-    <xacro:SimpleTransmissionEffort n="7" joint="joint_base_to_mors_1"/>
-    <xacro:SimpleTransmissionEffort n="8" joint="joint_base_to_mors_2"/>
+    <xacro:SimpleTransmissionPostion n="7" joint="joint_base_to_mors_1"/>
+    <xacro:SimpleTransmissionPostion n="8" joint="joint_base_to_mors_2"/>
     <!-- material -->
     <gazebo reference="base_gripper_1">
@@ -157,3 +146,3 @@
         <material>Gazebo/DarkGrey</material>
     </gazebo>
-</robot>
+</xml>
